File: assets/GnW_SD/GnW_SD.kicad_sch (KiCad schematic)
At the start: 7 parts, among them U2 RT9193-28GB

Commit message: Board cleanup & finish
Parts:
- C1, C2: LCSC (none) -> C28323
- C3: LCSC (none) -> C1804
- R1: LCSC (none) -> C25271
Changed lines of the file:
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@@
+			)
+		)
+		(property "LCSC" "C28323"
+			(at 169.418 123.444 0)
+			(effects
+				(font
+					(size 1.27 1.27)
+				)
+				(hide yes)
 			)
 		)
@@
 			)
 		)
+		(property "LCSC" "C28323"
+			(at 115.316 127.254 0)
+			(effects
+				(font
+					(size 1.27 1.27)
+				)
+				(hide yes)
+			)
+		)
 		(pin "2"
 		)
@@
 			)
 		)
+		(property "LCSC" "C25271"
+			(at 130.81 126.9999 0)
+			(effects
+				(font
+					(size 1.27 1.27)
+				)
+				(hide yes)
+			)
+		)
 		(pin "1"
 		)
@@
 			(effects
 				(font
+					(size 1.27 1.27)
+				)
+				(hide yes)
+			)
+		)
+		(property "LCSC" "C1804"
+			(at 160.274 123.444 0)
+			(effects
+				(font

Commit message: Update LCSC part numbers
Parts:
- C3: LCSC C1804 -> C1729
- R1: LCSC C25271 -> C25611
Changed lines of the file:
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@@
 			)
 		)
-		(property "LCSC" "C25271"
+		(property "LCSC" "C25611"
 			(at 130.81 126.9999 0)
 			(effects
@@
 			)
 		)
-		(property "LCSC" "C1804"
+		(property "LCSC" "C1729"
 			(at 160.274 123.444 0)
 			(effects
